Commit message: test: prove ground manipulator runtime

File: src/platform/ground_manipulator_runtime/urdf/ground_robot.urdf.xacro (robot description, xacro)
@@ -36,8 +36,8 @@
   <joint name="lidar_2d_joint" type="fixed">
     <parent link="base_link"/><child link="lidar_2d_link"/>
-    <origin xyz="-0.30 0 0.25" rpy="0 0 0"/>
+    <origin xyz="0.45 0 0.25" rpy="0 0 0"/>
   </joint>
   <gazebo reference="base_link">
-    <mu1>1.0</mu1><mu2>1.0</mu2>
+    <mu1>0.0</mu1><mu2>0.0</mu2>
   </gazebo>
   <gazebo reference="lidar_2d_link">

Commit message: refactor: expose driver-compatible sensor topics

File: src/platform/ground_manipulator_runtime/urdf/ground_robot.urdf.xacro (robot description, xacro)
@@ -38,6 +38,29 @@
     <origin xyz="0.45 0 0.25" rpy="0 0 0"/>
   </joint>
+  <link name="imu_link"/>
+  <joint name="imu_joint" type="fixed">
+    <parent link="base_link"/><child link="imu_link"/>
+    <origin xyz="0 0 0" rpy="0 0 0"/>
+  </joint>
   <gazebo reference="base_link">
     <mu1>0.0</mu1><mu2>0.0</mu2>
+  </gazebo>
+  <gazebo reference="imu_link">
+    <sensor name="bunker_imu" type="imu">
+      <always_on>true</always_on>
+      <update_rate>100.0</update_rate>
+      <visualize>false</visualize>
+      <plugin name="bunker_imu" filename="libgazebo_ros_imu_sensor.so">
+        <robotNamespace>/ground</robotNamespace>
+        <topicName>imu/data</topicName>
+        <bodyName>imu_link</bodyName>
+        <updateRateHZ>100.0</updateRateHZ>
+        <gaussianNoise>0.002</gaussianNoise>
+        <xyzOffset>0 0 0</xyzOffset>
+        <rpyOffset>0 0 0</rpyOffset>
+        <frameName>ground/imu_link</frameName>
+        <initialOrientationAsReference>false</initialOrientationAsReference>
+      </plugin>
+    </sensor>
   </gazebo>
   <gazebo reference="lidar_2d_link">
